File: hardware/pulsardew/pulsardew.kicad_sch (KiCad schematic)
At the start: 0 parts

Commit message: Add top-level schematic with MCU, USB-C, and hierarchical sheets
Top-level pulsardew.kicad_sch (A3) with:
- U1 STM32G0B1KBU6 (UFQFPN-32) with bypass/reset caps
- J1 USB-C 16P receptacle (GCT USB4105, C2927039) with 5.1k CC pulldowns
- 4× heater_channel.kicad_sch hierarchical sheets (PWM on PA0-PA3)
- 1× current_sense.kicad_sch hierarchical sheet (I2C on PB6/PB7)
- Net labels: USB_D+/D- (PA11/PA12), I2C_SDA/SCL, SWDIO/SWCLK, HTR_PWM0-3

Library additions:
- pulsarfab:STM32G0B1KBU6 symbol (from tsumikoro, LCSC C5159549)
- pulsarfab:UFQFPN-32 footprint (from tsumikoro)

Co-Authored-By: Claude Opus 4.6 (1M context) <noreply@anthropic.com>
Parts:
- added C1, C2: 100n, Capacitor_SMD:C_0402_1005Metric, symbol Device:C
- added J1: USB-C, Connector_USB:USB_C_Receptacle_GCT_USB4105-xx-A_16P_TopMnt_Horizontal, symbol Connector:USB_C_Receptacle_USB2.0_16P
- added R10, R11: 5.1k, Resistor_SMD:R_0402_1005Metric, symbol Device:R
- added U1: STM32G0B1KBU6, pulsarfab:UFQFPN-32, symbol pulsarfab:STM32G0B1KBU6
Connections:
- no-connect marks 0 -> 2
Other:
- added sheet Current Sense (current_sense.kicad_sch)
- added sheet Heater Ch0 (heater_channel.kicad_sch)
- added sheet Heater Ch1 (heater_channel.kicad_sch)
- added sheet Heater Ch2 (heater_channel.kicad_sch)
- added sheet Heater Ch3 (heater_channel.kicad_sch)
- note added: "PulsarDew — USB Dew Heater Controller"
- note added: "STM32G0B1KBU6 + USB-C + 4× heater channels + INA226 current sense + SHT40"
- company: PulsarFab -> (none)
- title: PulsarDew - USB Dew Heater Controller -> PulsarDew — USB Dew Heater Controller

Commit message: Add LDO, SHT40 sub-sheets, I2C pullups, power input with reverse polarity protection
New sub-sheets:
- ldo.kicad_sch: HT7333-A 30V→3.3V 250mA LDO (C347191) with 1µF 0402 in/out caps
- sht40.kicad_sch: Sensirion SHT40-AD1B-R2 temp/humidity (C2909890) with 100nF bypass

Top-level additions:
- R20/R21 4.7k 0402 I2C pull-ups on SDA/SCL to +3V3
- J2 DC barrel jack 2.0mm (C2880546) + J3 Phoenix COMBICON 2-pos (C480537)
- D10 SS54 Schottky reverse polarity diode (C22452, 40V/5A SMA)
- C10 470µF/25V electrolytic bulk cap after protection diode
- LDO and SHT40 hierarchical sheet references
- VIN_PROT net connecting protected input to LDO and heater channels

Full hierarchy: 8 sheets (top + 4 heater + current sense + LDO + SHT40)

Co-Authored-By: Claude Opus 4.6 (1M context) <noreply@anthropic.com>
Parts:
- added C10: 470u/25V, Capacitor_SMD:CP_Elec_8x10.5, symbol Device:C_Polarized
- added D10: SS54, Diode_SMD:D_SMA_Handsoldering, symbol Device:D_Schottky
- added J2: DC-005 2.0mm, Connector_BarrelJack:BarrelJack_GCT_DCJ200-10-A_Horizontal, symbol Connector:Barrel_Jack_Switch
- added J3: Phoenix 2-pos, Connector_Phoenix_MKDS:PhoenixContact_MKDS_3,2-5,08_1x02_P5.08mm_Horizontal, symbol Connector_Generic:Conn_01x02
- added R20, R21: 4.7k, Capacitor_SMD:C_0402_1005Metric, symbol Device:R
Other:
- added sheet LDO 3.3V (ldo.kicad_sch)
- added sheet SHT40 (sht40.kicad_sch)
- note added: "Power Input: 12-20V DC via barrel jack or Phoenix terminal"
- note added: "SS54 reverse polarity protection + 470µF bulk cap"
