File: hardware/pulsardew/current_sense.kicad_sch (KiCad schematic)
At the start: 3 parts, among them U1 INA226

Commit message: hardware: wire and verify the PulsarDew schematic hierarchy
Parts:
- renumbered C1 to C30, R1 to R30, U1 to U3
Connections:
- net GND: now also C30.2, U3.1 (A1), U3.2 (A0), U3.7 (GND)
- net SCL: now also U3.5 (SCL)
- net SDA: now also U3.4 (SDA)
- net VIN_IN: now also R30.1, U3.10 (Vin+)
- net VIN_OUT: now also R30.2, U3.8 (Vbus), U3.9 (Vin-)
- new net VDD: C30.1, U3.6 (VS)
Other:
- note added: "CURRENT MONITOR | INA226, I2C address 0x40"
- note added: "Route IN+ / IN- as Kelvin pairs directly to the shunt pads. VBUS senses the load side. A0 = A1 = GND. ALERT is unused. One monitor measures the combined heater current. 2 mOhm: 2.5 uV/LSB = 1.25 mA/LSB. ADC full scale is not the board current rating."
- note removed: "2mΩ shunt: 40A → 80mV, 50mA → 100µV. INA226 LSB=2.5µV → 1.25mA resolution."
- note removed: "I2C address 0x40 (A0=GND, A1=GND). Shares bus with SHT40 (0x44)."
- note removed: "Input Current Sense — INA226 High-Side Monitor"
- company: (none) -> PulsarFab
- title: Input Current Sense — INA226 High-Side Monitor -> PulsarDew - Input current monitor
