File: hardware/pulsardew/heater_channel.kicad_sch (KiCad schematic)
At the start: 7 parts, among them Q1 2N7002, Q2 AOD4184A

Commit message: hardware: wire and verify the PulsarDew schematic hierarchy
Parts:
- added J101: HEATER, TerminalBlock_Phoenix:TerminalBlock_Phoenix_MKDS-1,5-2-5.08_1x02_P5.08mm_Horizontal, symbol Connector_Generic:Conn_01x02
- Q101: renamed from Q1; symbol Transistor_FET:Q_NMOS_GDS -> Transistor_FET:2N7002
- renumbered D1 to D101, D2 to D102, Q2 to Q102, R1 to R101, R2 to R102, R3 to R103
Connections:
- net GND: now also D101.2 (A), D102.2 (A), Q101.2 (S), Q102.3 (S)
- net PWM: now also Q101.1 (G), R101.2
- net VIN: now also R102.1, J101.1 (Pin_1)
- new net: D101.1 (K), Q101.3 (D), R102.2, R103.1
- new net GATE_DRIVE: Q102.1 (G), R103.2
- new net HEATER_LOW: D102.1 (K), J101.2 (Pin_2), Q102.2 (D)
- new net VDD: R101.1
Other:
- note added: "HEATER DRIVER | Inverting, zener-clamped gate drive"
- note added: "PWM HIGH / high impedance with 3V3 present: heater OFF. PWM LOW: heater ON. Jx01 pin 1 = measured VIN; pin 2 = switched return. Do not bond pin 2 to ground. Default-off depends on 3V3: loss of logic power can turn the heater ON. Use slow PWM; verify switching loss, current limit and thermal margins on the bench."
- note removed: "Heater Channel — Zener-Clamped Level Shifter"
- note removed: "MCU PWM HIGH → Q1 ON → Gate LOW → Heater OFF (fail-safe default)"
- note removed: "MCU PWM LOW → Q1 OFF → Gate → 12V (clamped) → Heater ON"
- company: (none) -> PulsarFab
- title: Dew Heater Channel — Zener-Clamped Gate Drive -> PulsarDew - Heater driver (active-low PWM)
