File: hardware/pulsardew/ldo.kicad_sch (KiCad schematic)
At the start: 3 parts, among them U1 HT7333-A

Commit message: hardware: wire and verify the PulsarDew schematic hierarchy
Parts:
- added C22: 100n / 50V, Capacitor_SMD:C_0603_1608Metric, symbol Device:C
- added C23: 100n / 10V, Capacitor_SMD:C_0402_1005Metric, symbol Device:C
- C20: renamed from C1; value 1u -> 10u / 50V; footprint Capacitor_SMD:C_0402_1005Metric -> Capacitor_SMD:C_1210_3225Metric
- C21: renamed from C2; value 1u -> 10u / 10V; footprint Capacitor_SMD:C_0402_1005Metric -> Capacitor_SMD:C_0805_2012Metric
- U2: renamed from U1; value HT7333-A -> HT7333-1; symbol Regulator_Linear:L78L33_SOT89 -> pulsarfab:HT7333-1; LCSC C347191 -> (none); MPN HT7333-A -> HT7333-1; Manufacturer (none) -> Holtek
Connections:
- net GND: now also C20.2, C21.2, U2.1 (GND), C22.2, C23.2
- net VIN: now also C20.1, U2.2 (VIN), C22.1
- new net VDD: C21.1, C23.1, U2.3 (VOUT)
Other:
- note added: "LOGIC SUPPLY | HT7333-1, 30 V input rating"
- note added: "SOT-89 pinout: 1 GND, 2 VIN (tab), 3 VOUT. Use HT7333-1, not the 12 V HT7333 / 73xx-A part. Confirm exact orderable part before BOM release. 10 uF + 100 nF at input/output per Holtek application circuit; allow for DC-bias derating. Check LDO dissipation: (VIN - 3.3 V) x ILOGIC. The 250 mA headline is not a thermal allowance."
- note removed: "3.3V LDO — HT7333-A (30V max input, 250mA)"
- company: (none) -> PulsarFab
- title: 3.3V LDO — HT7333-A -> PulsarDew - 3.3V logic supply
