File: hardware/pulsardew/sht40.kicad_sch (KiCad schematic)
At the start: 2 parts, among them U1 SHT40-AD1B

Commit message: hardware: wire and verify the PulsarDew schematic hierarchy
Parts:
- renumbered C1 to C40, U1 to U4
Connections:
- net GND: now also C40.2, U4.4 (VSS)
- net SCL: now also U4.2 (SCL)
- net SDA: now also U4.1 (SDA)
- new net VDD: C40.1, U4.3 (VDD)
Other:
- note added: "100 nF at VDD/VSS. I2C pull-ups are on the Controller sheet. Place the sensor away from the LDO, MOSFETs and heater power copper."
- note added: "AMBIENT SENSOR | SHT40-AD1B, I2C address 0x44"
- note removed: "Temperature/Humidity Sensor — SHT40 I2C (addr 0x44)"
- company: (none) -> PulsarFab
- title: Temperature/Humidity — SHT40 -> PulsarDew - Temperature and humidity
