File: hardware/pulsardew/controller.kicad_sch (KiCad schematic)
At the start: 12 parts, among them J1 USB-C, J4 SWD, U1 STM32G0B1KBU6

Commit message: hardware: floorplan PulsarDew and check schematic parity
Parts:
- U1: footprint pulsarfab:UFQFPN-32 -> Package_DFN_QFN:UFQFPN-32-1EP_5x5mm_P0.5mm_EP3.5x3.5mm
Changed lines of the file:
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@@
       (font
         (size 1.27 1.27))))
-  (property "Footprint" "pulsarfab:UFQFPN-32"
+  (property "Footprint" "Package_DFN_QFN:UFQFPN-32-1EP_5x5mm_P0.5mm_EP3.5x3.5mm"
     (at 99.06 88.9 0.0)
     (effects

Commit message: Match PulsarDew connector sourcing to reviewed footprints
Parts:
- J1: LCSC C2927039 -> C3020560; MPN USB-TYPE-C-019 -> USB4105-GF-A; Manufacturer (none) -> GCT
Changed lines of the file:
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@@
         (size 1.27 1.27))
       (hide yes)))
-  (property "Datasheet" "https://www.usb.org/sites/default/files/documents/usb_type-c.zip"
+  (property "Datasheet" "https://gct.co/files/drawings/usb4105.pdf"
     (at 190.5 66.04 0.0)
     (effects
@@
         (size 1.27 1.27))
       (hide yes)))
-  (property "LCSC" "C2927039"
+  (property "LCSC" "C3020560"
     (at 190.5 66.04 0.0)
     (effects
@@
         (size 1.27 1.27))
       (hide yes)))
-  (property "MPN" "USB-TYPE-C-019"
+  (property "MPN" "USB4105-GF-A"
     (at 190.5 66.04 0.0)
     (effects
@@
       (path "/4235aaa6-671a-4985-9062-abb1f1decfe0/776ed70f-80c6-53e9-9e99-1ad3c8b58863"
         (reference "J1")
-        (unit 1)))))
+        (unit 1))))(property "Manufacturer" "GCT"
+  (at 190.5 66.04 0.0)
+  (effects
+    (font
+      (size 1.27 1.27))
+    (hide yes)))
+	)
 (symbol
   (lib_id "Device:R")

Commit message: Use stocked HRO USB-C sockets on PulsarPower and PulsarDew
Parts:
- J1: footprint Connector_USB:USB_C_Receptacle_GCT_USB4105-xx-A_16P_TopMnt_Horizontal -> pulsarfab:USB_C_HRO_TYPE-C-31-M-12; LCSC C3020560 -> C165948; MPN USB4105-GF-A -> TYPE-C-31-M-12; Manufacturer GCT -> Korean Hroparts Elec
Changed lines of the file:
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@@
       (font
         (size 1.27 1.27))))
-  (property "Footprint" "Connector_USB:USB_C_Receptacle_GCT_USB4105-xx-A_16P_TopMnt_Horizontal"
+  (property "Footprint" "pulsarfab:USB_C_HRO_TYPE-C-31-M-12"
     (at 190.5 66.04 0.0)
     (effects
@@
         (size 1.27 1.27))
       (hide yes)))
-  (property "Datasheet" "https://gct.co/files/drawings/usb4105.pdf"
+  (property "Datasheet" "https://datasheet.lcsc.com/datasheet/pdf/9e56b777c022540fcce7c7f67825f55e.pdf?productCode=C165948"
     (at 190.5 66.04 0.0)
     (effects
@@
         (size 1.27 1.27))
       (hide yes)))
-  (property "LCSC" "C3020560"
+  (property "LCSC" "C165948"
     (at 190.5 66.04 0.0)
     (effects
@@
         (size 1.27 1.27))
       (hide yes)))
-  (property "MPN" "USB4105-GF-A"
+  (property "MPN" "TYPE-C-31-M-12"
     (at 190.5 66.04 0.0)
     (effects
@@
       (path "/4235aaa6-671a-4985-9062-abb1f1decfe0/776ed70f-80c6-53e9-9e99-1ad3c8b58863"
         (reference "J1")
-        (unit 1))))(property "Manufacturer" "GCT"
+        (unit 1))))(property "Manufacturer" "Korean Hroparts Elec"
   (at 190.5 66.04 0.0)
   (effects
