File: hardware/pulsardew/pulsardew.kicad_pcb (KiCad board)
At the start: 2 copper layers, 0 parts

Commit message: hardware: floorplan PulsarDew and check schematic parity
Parts:
- added C1: 100n, Capacitor_SMD:C_0402_1005Metric, F.Cu at (132.0, 70.4)
- added C10: 470u/25V, Capacitor_SMD:CP_Elec_8x10.5, F.Cu at (78.0, 85.0)
- added C2: 100n, Capacitor_SMD:C_0402_1005Metric, F.Cu at (131.0, 73.0)
- added C20: 10u / 50V, Capacitor_SMD:C_1210_3225Metric, F.Cu at (74.0, 63.0)
- added C21: 10u / 10V, Capacitor_SMD:C_0805_2012Metric, F.Cu at (76.0, 66.0)
- added C22: 100n / 50V, Capacitor_SMD:C_0603_1608Metric, F.Cu at (75.0, 58.5)
- added C23: 100n / 10V, Capacitor_SMD:C_0402_1005Metric, F.Cu at (80.0, 65.0)
- added C3: 4.7u / 10V, Capacitor_SMD:C_0402_1005Metric, F.Cu at (134.5, 71.0)
- added C30: 100n, Capacitor_SMD:C_0402_1005Metric, F.Cu at (94.3, 82.5)
- added C40: 100n, Capacitor_SMD:C_0402_1005Metric, F.Cu at (145.5, 66.0)
- added D10: SS54, Diode_SMD:D_SMA_Handsoldering, F.Cu at (73.0, 74.0)
- added D101: BZT52C12 12V, Diode_SMD:D_SOD-123, F.Cu at (74.0, 113.0)
- added D102: SMBJ20A, Diode_SMD:D_SMB_Handsoldering, F.Cu at (83.0, 115.8)
- added D201: BZT52C12 12V, Diode_SMD:D_SOD-123, F.Cu at (92.0, 113.0)
- added D202: SMBJ20A, Diode_SMD:D_SMB_Handsoldering, F.Cu at (101.0, 115.8)
- added D301: BZT52C12 12V, Diode_SMD:D_SOD-123, F.Cu at (110.0, 113.0)
- added D302: SMBJ20A, Diode_SMD:D_SMB_Handsoldering, F.Cu at (119.0, 115.8)
- added D401: BZT52C12 12V, Diode_SMD:D_SOD-123, F.Cu at (128.0, 113.0)
- added D402: SMBJ20A, Diode_SMD:D_SMB_Handsoldering, F.Cu at (137.0, 115.8)
- added H1: M3, MountingHole_3.2mm_M3, F.Cu at (54.0, 54.0)
- added H2: M3, MountingHole_3.2mm_M3, F.Cu at (146.0, 54.0)
- added H3: M3, MountingHole_3.2mm_M3, F.Cu at (54.0, 126.0)
- added H4: M3, MountingHole_3.2mm_M3, F.Cu at (146.0, 126.0)
- added J1: USB-C, Connector_USB:USB_C_Receptacle_GCT_USB4105-xx-A_16P_TopMnt_Horizontal, F.Cu at (132.0, 54.0)
- added J101: HEATER, TerminalBlock_Phoenix:TerminalBlock_Phoenix_MKDS-1,5-2-5.08_1x02_P5.08mm_Horizontal, F.Cu at (80.0, 124.4)
- added J2: DC-005 2.0mm, Connector_BarrelJack:BarrelJack_GCT_DCJ200-10-A_Horizontal, F.Cu at (64.5, 71.0)
- added J201: HEATER, TerminalBlock_Phoenix:TerminalBlock_Phoenix_MKDS-1,5-2-5.08_1x02_P5.08mm_Horizontal, F.Cu at (98.0, 124.4)
- added J3: Phoenix 2-pos, TerminalBlock_Phoenix:TerminalBlock_Phoenix_MKDS-1,5-2-5.08_1x02_P5.08mm_Horizontal, F.Cu at (55.9, 90.0)
- added J301: HEATER, TerminalBlock_Phoenix:TerminalBlock_Phoenix_MKDS-1,5-2-5.08_1x02_P5.08mm_Horizontal, F.Cu at (116.0, 124.4)
- added J4: SWD, Connector_PinHeader_2.54mm:PinHeader_1x05_P2.54mm_Vertical, F.Cu at (115.0, 61.0)
- added J401: HEATER, TerminalBlock_Phoenix:TerminalBlock_Phoenix_MKDS-1,5-2-5.08_1x02_P5.08mm_Horizontal, F.Cu at (134.0, 124.4)
- added Q101: 2N7002, Package_TO_SOT_SMD:SOT-23, F.Cu at (75.5, 108.0)
- added Q102: AOD4184A, Package_TO_SOT_SMD:TO-252-2, F.Cu at (81.0, 107.0)
- added Q201: 2N7002, Package_TO_SOT_SMD:SOT-23, F.Cu at (93.5, 108.0)
- added Q202: AOD4184A, Package_TO_SOT_SMD:TO-252-2, F.Cu at (99.0, 107.0)
- added Q301: 2N7002, Package_TO_SOT_SMD:SOT-23, F.Cu at (111.5, 108.0)
- added Q302: AOD4184A, Package_TO_SOT_SMD:TO-252-2, F.Cu at (117.0, 107.0)
- added Q401: 2N7002, Package_TO_SOT_SMD:SOT-23, F.Cu at (129.5, 108.0)
- added Q402: AOD4184A, Package_TO_SOT_SMD:TO-252-2, F.Cu at (135.0, 107.0)
- added R10: 5.1k, Resistor_SMD:R_0402_1005Metric, F.Cu at (129.0, 60.5)
- added R101: 100k, Resistor_SMD:R_0402_1005Metric, F.Cu at (72.5, 106.0)
- added R102: 10k, Resistor_SMD:R_0402_1005Metric, F.Cu at (74.0, 103.5)
- added R103: 47, Resistor_SMD:R_0402_1005Metric, F.Cu at (77.0, 115.0)
- added R11: 5.1k, Resistor_SMD:R_0402_1005Metric, F.Cu at (135.0, 60.5)
- added R12: 100k, Resistor_SMD:R_0402_1005Metric, F.Cu at (137.0, 65.5)
- added R13: 100k, Resistor_SMD:R_0402_1005Metric, F.Cu at (137.0, 68.0)
- added R20: 4.7k, Resistor_SMD:R_0402_1005Metric, F.Cu at (127.0, 64.0)
- added R201: 100k, Resistor_SMD:R_0402_1005Metric, F.Cu at (90.5, 106.0)
- added R202: 10k, Resistor_SMD:R_0402_1005Metric, F.Cu at (92.0, 103.5)
- added R203: 47, Resistor_SMD:R_0402_1005Metric, F.Cu at (95.0, 115.0)
- added R21: 4.7k, Resistor_SMD:R_0402_1005Metric, F.Cu at (127.0, 66.0)
- added R30: 2m, Resistor_SMD:R_2512_6332Metric, F.Cu at (90.0, 78.0)
- added R301: 100k, Resistor_SMD:R_0402_1005Metric, F.Cu at (108.5, 106.0)
- added R302: 10k, Resistor_SMD:R_0402_1005Metric, F.Cu at (110.0, 103.5)
- added R303: 47, Resistor_SMD:R_0402_1005Metric, F.Cu at (113.0, 115.0)
- added R401: 100k, Resistor_SMD:R_0402_1005Metric, F.Cu at (126.5, 106.0)
- added R402: 10k, Resistor_SMD:R_0402_1005Metric, F.Cu at (128.0, 103.5)
- added R403: 47, Resistor_SMD:R_0402_1005Metric, F.Cu at (131.0, 115.0)
- added U1: STM32G0B1KBU6, Package_DFN_QFN:UFQFPN-32-1EP_5x5mm_P0.5mm_EP3.5x3.5mm, F.Cu at (132.0, 66.0)
- added U2: HT7333-1, Package_TO_SOT_SMD:SOT-89-3, F.Cu at (80.0, 61.0)
- added U3: INA226, Package_SO:TSSOP-10_3x3mm_P0.5mm, F.Cu at (90.0, 84.0)
- added U4: SHT40-AD1B, Sensor_Humidity:Sensirion_DFN-4_1.5x1.5mm_P0.8mm_SHT4x_NoCentralPad, F.Cu at (143.0, 66.0)
Other:
- board outline added: 100 x 80 mm
- board text added: "DC IN 12-20V"
- board text added: "FLOORPLAN - UNROUTED"
- board text added: "HEATER 0"
- board text added: "HEATER 1"
- board text added: "HEATER 2"
- board text added: "HEATER 3"
- board text added: "Kelvin sense at R30 pads"
- board text added: "ONE INPUT ONLY"
- board text added: "Power corridor: input > shunt > heater rail"
- board text added: "PulsarDew 0.3"
- board text added: "SHT40"
- board text added: "SWD"
- board text added: "USB"

Commit message: Match PulsarDew connector sourcing to reviewed footprints
Parts:
- J2: value DC-005 2.0mm -> DCJ200 / 2.0mm / 5A
Changed lines of the file:
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@@
 			)
 		)
-		(property "Datasheet" "https://www.usb.org/sites/default/files/documents/usb_type-c.zip"
+		(property "Datasheet" "https://gct.co/files/drawings/usb4105.pdf"
 			(at 0 0 180)
 			(unlocked yes)
@@
 			)
 		)
-		(property "LCSC" "C2927039"
+		(property "LCSC" "C3020560"
 			(at 0 0 180)
 			(unlocked yes)
@@
 			)
 		)
-		(property "MPN" "USB-TYPE-C-019"
+		(property "MPN" "USB4105-GF-A"
 			(at 0 0 180)
 			(unlocked yes)
@@
 					(size 1 1)
 					(thickness 0.15)
+				)
+			)
+		)
+		(property "Manufacturer" "GCT"
+			(at 0 0 0)
+			(layer "F.SilkS")
+			(hide yes)
+			(effects
+				(font
+					(size 1.27 1.27)
 				)
 			)
@@
 			)
 		)
-		(property "Value" "DC-005 2.0mm"
+		(property "Value" "DCJ200 / 2.0mm / 5A"
 			(at 0 15.5 270)
 			(layer "F.Fab")
@@
 			)
 		)
-		(property "Datasheet" ""
+		(property "Datasheet" "https://gct.co/files/drawings/dcj200.pdf"
 			(at 0 0 270)
 			(unlocked yes)
@@
 			)
 		)
-		(property "LCSC" "C2880546"
+		(property "LCSC" "C5280493"
 			(at 0 0 270)
 			(unlocked yes)
@@
 			)
 		)
-		(property "MPN" "DC-005K-5A-2.0"
+		(property "MPN" "DCJ200-10-A-K1-K"
 			(at 0 0 270)
 			(unlocked yes)
@@
 				)
 			)
+		)
+		(property "Manufacturer" "GCT"
+			(at 0 0 0)
+			(layer "F.SilkS")
+			(hide yes)
+			(effects
+				(font
+					(size 1.27 1.27)
+				)
+			)

Commit message: Use stocked HRO USB-C sockets on PulsarPower and PulsarDew
Parts:
- J1: footprint Connector_USB:USB_C_Receptacle_GCT_USB4105-xx-A_16P_TopMnt_Horizontal -> pulsarfab:USB_C_HRO_TYPE-C-31-M-12
- moved J1 0.81 mm to (132.0, 53.2)

Commit message: Use owned XKB barrel sockets and evaluate LMR51610 commonality
Parts:
- J2: value DCJ200 / 2.0mm / 5A -> XKB DC-005K / 5A; footprint Connector_BarrelJack:BarrelJack_GCT_DCJ200-10-A_Horizontal -> pulsarfab:BarrelJack_XKB_DC-005K-5A_Edge
Connections:
- J2 pad 3: unconnected-(J2-Pad3) -> /GND
