File: hardware/pulsardewhub/heaters.kicad_sch (KiCad schematic)
At the start: 20 parts, among them J51 HEATER 1, J61 HEATER 2, Q51 AOD4184A, Q61 AOD4184A, U50 TC4427AVOA713, U51 INA226

Commit message: Reduce PulsarPower power-path cost while retaining current monitoring
Other:
- title: PulsarDew Hub - Two default-off heater outputs -> PulsarPower - Two default-off heater outputs
Changed lines of the file:
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@@
 (kicad_sch (version 20260306) (generator "eeschema") (generator_version "10.0") (paper "A3")
-(title_block (title "PulsarDew Hub - Two default-off heater outputs") (date "2026-10-03") (rev "0.2-draft") (company "PulsarFab"))
+(title_block (title "PulsarPower - Two default-off heater outputs") (date "2026-10-03") (rev "0.3-draft") (company "PulsarFab"))
 (text "HEATERS | active-high PWM, 5 V gate drive, resistive loads only" (at 20.3200 16.5100 0) (effects (font (size 2 2)) (justify left top)))
 (hierarchical_label "VIN" (shape input) (at 25.4000 40.6400 0) (effects (font (size 1.27 1.27)) (justify left bottom)))
