File: hardware/pulsardewhub/pulsardewhub.kicad_sch (KiCad schematic)
At the start: 0 parts

Commit message: Use TPS259827 high-side switches for 12–18 V DC outlets
Other:
- sheet Controller ports: added DC_PG1, DC_PG2, DC_PG3, DC_PG4; removed DC_FLT1, DC_FLT2, DC_FLT3, DC_FLT4
- sheet DC outlet 1 ports: added PGOOD; removed FAULT
- sheet DC outlet 2 ports: added PGOOD; removed FAULT
- sheet DC outlet 3 ports: added PGOOD; removed FAULT
- sheet DC outlet 4 ports: added PGOOD; removed FAULT
- note added: "RATINGS TO VALIDATE 12-18 V nominal input 4 x 5 A DC outlet targets 2 x 5 A heater targets 25 A shared XT60 budget 3.5 A continuous barrel budget USB: 500 mA per port No PWM on DC outlets"
- note removed: "RATINGS TO VALIDATE 12-20 V nominal input 4 x 5 A DC outlet targets 2 x 5 A heater targets 25 A shared XT60 budget 3.5 A continuous barrel budget USB: 500 mA per port No PWM on DC outlets"
Changed lines of the file:
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@@
 (kicad_sch (version 20260306) (generator "eeschema") (generator_version "10.0") (paper "A2")
-(title_block (title "PulsarDew Hub - System interconnect") (date "2026-10-03") (rev "0.1-draft") (company "PulsarFab"))
+(title_block (title "PulsarDew Hub - System interconnect") (date "2026-10-03") (rev "0.2-draft") (company "PulsarFab"))
 (text "PULSARDEW HUB | 2 heaters + 4 monitored DC outlets + 4 USB 2.0 ports" (at 20.3200 16.5100 0) (effects (font (size 2.5 2.5)) (justify left top)))
 (text "PROTOTYPE FLOORPLAN — routing, full-load thermal validation and new firmware are still required." (at 20.3200 24.1300 0) (effects (font (size 1.5 1.5)) (justify left top)))
@@
 (label "DC_EN1"  (at 208.2800 99.0600 180) (effects (font (size 1.27 1.27)) (justify right bottom)))
 (label "IMON1"  (at 208.2800 104.1400 180) (effects (font (size 1.27 1.27)) (justify right bottom)))
-(label "DC_FLT1"  (at 208.2800 109.2200 180) (effects (font (size 1.27 1.27)) (justify right bottom)))
+(label "DC_PG1"  (at 208.2800 109.2200 180) (effects (font (size 1.27 1.27)) (justify right bottom)))
 (label "DC_EN2"  (at 208.2800 114.3000 180) (effects (font (size 1.27 1.27)) (justify right bottom)))
 (label "IMON2"  (at 208.2800 119.3800 180) (effects (font (size 1.27 1.27)) (justify right bottom)))
-(label "DC_FLT2"  (at 208.2800 124.4600 180) (effects (font (size 1.27 1.27)) (justify right bottom)))
+(label "DC_PG2"  (at 208.2800 124.4600 180) (effects (font (size 1.27 1.27)) (justify right bottom)))
 (label "DC_EN3"  (at 208.2800 129.5400 180) (effects (font (size 1.27 1.27)) (justify right bottom)))
 (label "IMON3"  (at 208.2800 134.6200 180) (effects (font (size 1.27 1.27)) (justify right bottom)))
-(label "DC_FLT3"  (at 208.2800 139.7000 180) (effects (font (size 1.27 1.27)) (justify right bottom)))
+(label "DC_PG3"  (at 208.2800 139.7000 180) (effects (font (size 1.27 1.27)) (justify right bottom)))
 (label "DC_EN4"  (at 208.2800 144.7800 180) (effects (font (size 1.27 1.27)) (justify right bottom)))
 (label "IMON4"  (at 208.2800 149.8600 180) (effects (font (size 1.27 1.27)) (justify right bottom)))
-(label "DC_FLT4"  (at 208.2800 154.9400 180) (effects (font (size 1.27 1.27)) (justify right bottom)))
+(label "DC_PG4"  (at 208.2800 154.9400 180) (effects (font (size 1.27 1.27)) (justify right bottom)))
 (sheet
   (at 220.98 43.18)
@@
       (justify left))
 )
-  (pin "DC_FLT1" input
+  (pin "DC_PG1" input
     (at 220.98 109.22 180.0)
     (effects
@@
       (justify left))
 )
-  (pin "DC_FLT2" input
+  (pin "DC_PG2" input
     (at 220.98 124.46 180.0)
     (effects
@@
       (justify left))
 )
-  (pin "DC_FLT3" input
+  (pin "DC_PG3" input
     (at 220.98 139.7 180.0)
     (effects
@@
       (justify left))
 )
-  (pin "DC_FLT4" input
+  (pin "DC_PG4" input
     (at 220.98 154.94 180.0)
     (effects
@@
 (label "DC_EN1"  (at 363.2200 68.5800 180) (effects (font (size 1.27 1.27)) (justify right bottom)))
 (label "IMON1"  (at 363.2200 73.6600 180) (effects (font (size 1.27 1.27)) (justify right bottom)))
-(label "DC_FLT1"  (at 363.2200 78.7400 180) (effects (font (size 1.27 1.27)) (justify right bottom)))
+(label "DC_PG1"  (at 363.2200 78.7400 180) (effects (font (size 1.27 1.27)) (justify right bottom)))
 (sheet
   (at 375.92 43.18)
@@
       (justify left))
 )
-  (pin "FAULT" output
+  (pin "PGOOD" output
     (at 375.92 78.74 180.0)
     (effects
@@
 (label "DC_EN2"  (at 363.2200 149.8600 180) (effects (font (size 1.27 1.27)) (justify right bottom)))
 (label "IMON2"  (at 363.2200 154.9400 180) (effects (font (size 1.27 1.27)) (justify right bottom)))
-(label "DC_FLT2"  (at 363.2200 160.0200 180) (effects (font (size 1.27 1.27)) (justify right bottom)))
+(label "DC_PG2"  (at 363.2200 160.0200 180) (effects (font (size 1.27 1.27)) (justify right bottom)))
 (sheet
   (at 375.92 124.46)
@@
       (justify left))
 )
-  (pin "FAULT" output
+  (pin "PGOOD" output
     (at 375.92 160.02 180.0)
     (effects
@@
 (label "DC_EN3"  (at 363.2200 231.1400 180) (effects (font (size 1.27 1.27)) (justify right bottom)))
 (label "IMON3"  (at 363.2200 236.2200 180) (effects (font (size 1.27 1.27)) (justify right bottom)))
-(label "DC_FLT3"  (at 363.2200 241.3000 180) (effects (font (size 1.27 1.27)) (justify right bottom)))
+(label "DC_PG3"  (at 363.2200 241.3000 180) (effects (font (size 1.27 1.27)) (justify right bottom)))
 (sheet
   (at 375.92 205.74)
@@
       (justify left))
 )
-  (pin "FAULT" output
+  (pin "PGOOD" output
     (at 375.92 241.3 180.0)
     (effects
@@
 (label "DC_EN4"  (at 363.2200 312.4200 180) (effects (font (size 1.27 1.27)) (justify right bottom)))
 (label "IMON4"  (at 363.2200 317.5000 180) (effects (font (size 1.27 1.27)) (justify right bottom)))
-(label "DC_FLT4"  (at 363.2200 322.5800 180) (effects (font (size 1.27 1.27)) (justify right bottom)))
+(label "DC_PG4"  (at 363.2200 322.5800 180) (effects (font (size 1.27 1.27)) (justify right bottom)))
 (sheet
   (at 375.92 287.02)
@@
       (justify left))
 )
-  (pin "FAULT" output
+  (pin "PGOOD" output
     (at 375.92 322.58 180.0)
     (effects
@@
       (path "/e52b73dc-d0d2-4d83-a7ea-224e97decc28"
         (page "14")))))
-(text "RATINGS TO VALIDATE\n12-20 V nominal input\n4 x 5 A DC outlet targets\n2 x 5 A heater targets\n25 A shared XT60 budget\n3.5 A continuous barrel budget\nUSB: 500 mA per port\nNo PWM on DC outlets" (at 25.4000 281.9400 0) (effects (font (size 1.5 1.5)) (justify left top)))
+(text "RATINGS TO VALIDATE\n12-18 V nominal input\n4 x 5 A DC outlet targets\n2 x 5 A heater targets\n25 A shared XT60 budget\n3.5 A continuous barrel budget\nUSB: 500 mA per port\nNo PWM on DC outlets" (at 25.4000 281.9400 0) (effects (font (size 1.5 1.5)) (justify left top)))
 (text "Same ground throughout.\nHigh-current and USB return paths\nare separated by placement.\nDo not backfeed DC outputs." (at 25.4000 353.0600 0) (effects (font (size 1.27 1.27)) (justify left top)))
 (wire (pts (xy 17.7800 58.4200) (xy 17.7800 119.3800)) (stroke (width 0) (type default)))

Commit message: Reduce PulsarPower power-path cost while retaining current monitoring
Other:
- added sheet DC protection (dc_protection.kicad_sch)
- note added: "PULSARPOWER | 2 heaters + 4 monitored DC outlets + 4 USB 2.0 ports"
- note removed: "PULSARDEW HUB | 2 heaters + 4 monitored DC outlets + 4 USB 2.0 ports"
- title: PulsarDew Hub - System interconnect -> PulsarPower - System interconnect
Changed lines of the file:
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@@
 (kicad_sch (version 20260306) (generator "eeschema") (generator_version "10.0") (paper "A2")
-(title_block (title "PulsarDew Hub - System interconnect") (date "2026-10-03") (rev "0.2-draft") (company "PulsarFab"))
-(text "PULSARDEW HUB | 2 heaters + 4 monitored DC outlets + 4 USB 2.0 ports" (at 20.3200 16.5100 0) (effects (font (size 2.5 2.5)) (justify left top)))
+(title_block (title "PulsarPower - System interconnect") (date "2026-10-03") (rev "0.3-draft") (company "PulsarFab"))
+(text "PULSARPOWER | 2 heaters + 4 monitored DC outlets + 4 USB 2.0 ports" (at 20.3200 16.5100 0) (effects (font (size 2.5 2.5)) (justify left top)))
 (text "PROTOTYPE FLOORPLAN — routing, full-load thermal validation and new firmware are still required." (at 20.3200 24.1300 0) (effects (font (size 1.5 1.5)) (justify left top)))
 (label "VIN"  (at 40.6400 53.3400 180) (effects (font (size 1.27 1.27)) (justify right bottom)))
@@
 (label "V3"  (at 363.2200 58.4200 180) (effects (font (size 1.27 1.27)) (justify right bottom)))
 (label "GND"  (at 363.2200 63.5000 180) (effects (font (size 1.27 1.27)) (justify right bottom)))
-(label "DC_EN1"  (at 363.2200 68.5800 180) (effects (font (size 1.27 1.27)) (justify right bottom)))
+(label "DC_SAFE1"  (at 363.2200 68.5800 180) (effects (font (size 1.27 1.27)) (justify right bottom)))
 (label "IMON1"  (at 363.2200 73.6600 180) (effects (font (size 1.27 1.27)) (justify right bottom)))
 (label "DC_PG1"  (at 363.2200 78.7400 180) (effects (font (size 1.27 1.27)) (justify right bottom)))
@@
 (label "V3"  (at 363.2200 139.7000 180) (effects (font (size 1.27 1.27)) (justify right bottom)))
 (label "GND"  (at 363.2200 144.7800 180) (effects (font (size 1.27 1.27)) (justify right bottom)))
-(label "DC_EN2"  (at 363.2200 149.8600 180) (effects (font (size 1.27 1.27)) (justify right bottom)))
+(label "DC_SAFE2"  (at 363.2200 149.8600 180) (effects (font (size 1.27 1.27)) (justify right bottom)))
 (label "IMON2"  (at 363.2200 154.9400 180) (effects (font (size 1.27 1.27)) (justify right bottom)))
 (label "DC_PG2"  (at 363.2200 160.0200 180) (effects (font (size 1.27 1.27)) (justify right bottom)))
@@
 (label "V3"  (at 363.2200 220.9800 180) (effects (font (size 1.27 1.27)) (justify right bottom)))
 (label "GND"  (at 363.2200 226.0600 180) (effects (font (size 1.27 1.27)) (justify right bottom)))
-(label "DC_EN3"  (at 363.2200 231.1400 180) (effects (font (size 1.27 1.27)) (justify right bottom)))
+(label "DC_SAFE3"  (at 363.2200 231.1400 180) (effects (font (size 1.27 1.27)) (justify right bottom)))
 (label "IMON3"  (at 363.2200 236.2200 180) (effects (font (size 1.27 1.27)) (justify right bottom)))
 (label "DC_PG3"  (at 363.2200 241.3000 180) (effects (font (size 1.27 1.27)) (justify right bottom)))
@@
 (label "V3"  (at 363.2200 302.2600 180) (effects (font (size 1.27 1.27)) (justify right bottom)))
 (label "GND"  (at 363.2200 307.3400 180) (effects (font (size 1.27 1.27)) (justify right bottom)))
-(label "DC_EN4"  (at 363.2200 312.4200 180) (effects (font (size 1.27 1.27)) (justify right bottom)))
+(label "DC_SAFE4"  (at 363.2200 312.4200 180) (effects (font (size 1.27 1.27)) (justify right bottom)))
 (label "IMON4"  (at 363.2200 317.5000 180) (effects (font (size 1.27 1.27)) (justify right bottom)))
 (label "DC_PG4"  (at 363.2200 322.5800 180) (effects (font (size 1.27 1.27)) (justify right bottom)))
@@
       (path "/e52b73dc-d0d2-4d83-a7ea-224e97decc28"
         (page "14")))))
+(label "VIN"  (at 208.2800 345.4400 180) (effects (font (size 1.27 1.27)) (justify right bottom)))
+(label "V3"  (at 208.2800 350.5200 180) (effects (font (size 1.27 1.27)) (justify right bottom)))
+(label "GND"  (at 208.2800 355.6000 180) (effects (font (size 1.27 1.27)) (justify right bottom)))
+(label "DC_EN1"  (at 208.2800 360.6800 180) (effects (font (size 1.27 1.27)) (justify right bottom)))
+(label "DC_EN2"  (at 208.2800 365.7600 180) (effects (font (size 1.27 1.27)) (justify right bottom)))
+(label "DC_EN3"  (at 208.2800 370.8400 180) (effects (font (size 1.27 1.27)) (justify right bottom)))
+(label "DC_EN4"  (at 208.2800 375.9200 180) (effects (font (size 1.27 1.27)) (justify right bottom)))
+(label "DC_SAFE1"  (at 208.2800 381.0000 180) (effects (font (size 1.27 1.27)) (justify right bottom)))
+(label "DC_SAFE2"  (at 208.2800 386.0800 180) (effects (font (size 1.27 1.27)) (justify right bottom)))
+(label "DC_SAFE3"  (at 208.2800 391.1600 180) (effects (font (size 1.27 1.27)) (justify right bottom)))
+(label "DC_SAFE4"  (at 208.2800 396.2400 180) (effects (font (size 1.27 1.27)) (justify right bottom)))
+(sheet
+  (at 220.98 335.28)
+  (size 76.2 71.12)
+  (stroke
+    (width 0.1524)
+    (type default))
+  (fill
+    (color 0 0 0 0))
+  (property "Sheetname" "DC protection"
+    (at 220.98 332.74 0.0)
+    (effects
+      (font
+        (size 1.27 1.27))
+      (justify left)))
+  (property "Sheetfile" "dc_protection.kicad_sch"
+    (at 220.98 408.94 0.0)
+    (effects
+      (font
+        (size 1.27 1.27))
+      (justify left)))
+  (pin "VIN" input
+    (at 220.98 345.44 180.0)
+    (effects
+      (font
+        (size 1.27 1.27))
+      (justify left))
+)
+  (pin "V3" input
+    (at 220.98 350.52 180.0)
+    (effects
+      (font
+        (size 1.27 1.27))
+      (justify left))
+)
+  (pin "GND" input
+    (at 220.98 355.6 180.0)
+    (effects
+      (font
+        (size 1.27 1.27))
+      (justify left))
+)
+  (pin "CMD1" input
+    (at 220.98 360.68 180.0)
+    (effects
+      (font
+        (size 1.27 1.27))
+      (justify left))
+)
+  (pin "CMD2" input
+    (at 220.98 365.76 180.0)
+    (effects
+      (font
+        (size 1.27 1.27))
+      (justify left))
+)
+  (pin "CMD3" input
+    (at 220.98 370.84 180.0)
+    (effects
+      (font
+        (size 1.27 1.27))
+      (justify left))
+)
+  (pin "CMD4" input
+    (at 220.98 375.92 180.0)
+    (effects
+      (font
+        (size 1.27 1.27))
+      (justify left))
+)
+  (pin "EN1" output
+    (at 220.98 381.0 180.0)
+    (effects
+      (font
+        (size 1.27 1.27))
+      (justify left))
+)
+  (pin "EN2" output
+    (at 220.98 386.08 180.0)
+    (effects
+      (font
+        (size 1.27 1.27))
+      (justify left))
+)
+  (pin "EN3" output
+    (at 220.98 391.16 180.0)
+    (effects
+      (font
+        (size 1.27 1.27))
+      (justify left))
+)
+  (pin "EN4" output
+    (at 220.98 396.24 180.0)
+    (effects
+      (font
+        (size 1.27 1.27))
+      (justify left))
+)
+  (instances
+    (project "pulsardewhub"
+      (path "/e52b73dc-d0d2-4d83-a7ea-224e97decc28"
+        (page "15")))))
 (text "RATINGS TO VALIDATE\n12-18 V nominal input\n4 x 5 A DC outlet targets\n2 x 5 A heater targets\n25 A shared XT60 budget\n3.5 A continuous barrel budget\nUSB: 500 mA per port\nNo PWM on DC outlets" (at 25.4000 281.9400 0) (effects (font (size 1.5 1.5)) (justify left top)))
 (text "Same ground throughout.\nHigh-current and USB return paths\nare separated by placement.\nDo not backfeed DC outputs." (at 25.4000 353.0600 0) (effects (font (size 1.27 1.27)) (justify left top)))
@@
 (wire (pts (xy 208.2800 297.1800) (xy 220.9800 297.1800)) (stroke (width 0) (type default)))
 (wire (pts (xy 208.2800 302.2600) (xy 220.9800 302.2600)) (stroke (width 0) (type default)))
+(wire (pts (xy 208.2800 345.4400) (xy 220.9800 345.4400)) (stroke (width 0) (type default)))
+(wire (pts (xy 208.2800 350.5200) (xy 220.9800 350.5200)) (stroke (width 0) (type default)))
+(wire (pts (xy 208.2800 355.6000) (xy 220.9800 355.6000)) (stroke (width 0) (type default)))
+(wire (pts (xy 208.2800 360.6800) (xy 220.9800 360.6800)) (stroke (width 0) (type default)))
+(wire (pts (xy 208.2800 365.7600) (xy 220.9800 365.7600)) (stroke (width 0) (type default)))
+(wire (pts (xy 208.2800 370.8400) (xy 220.9800 370.8400)) (stroke (width 0) (type default)))
+(wire (pts (xy 208.2800 375.9200) (xy 220.9800 375.9200)) (stroke (width 0) (type default)))
+(wire (pts (xy 208.2800 381.0000) (xy 220.9800 381.0000)) (stroke (width 0) (type default)))
+(wire (pts (xy 208.2800 386.0800) (xy 220.9800 386.0800)) (stroke (width 0) (type default)))
+(wire (pts (xy 208.2800 391.1600) (xy 220.9800 391.1600)) (stroke (width 0) (type default)))
+(wire (pts (xy 208.2800 396.2400) (xy 220.9800 396.2400)) (stroke (width 0) (type default)))
 (wire (pts (xy 363.2200 53.3400) (xy 375.9200 53.3400)) (stroke (width 0) (type default)))
 (wire (pts (xy 363.2200 58.4200) (xy 375.9200 58.4200)) (stroke (width 0) (type default)))
