File: hardware/pulsardewhub/usb_port.kicad_sch (KiCad schematic)
At the start: 8 parts, among them J501 USB-A / 500mA, U501 TPS2553DBV, U502 USBLC6-2SC6

Commit message: Use economical through-hole USB-A sockets for PulsarPower
Parts:
- J501: footprint pulsarfab:USB_A_GCT_USB1046_Edge -> pulsarfab:USB_A_SHOUHAN_AF90ZJWG_THT; LCSC C6307429 -> C456019; MPN USB1046-GF-0190-L-B-A -> AF 90 ZJWG; Manufacturer Global Connector Technology -> SHOU HAN
Changed lines of the file:
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@@
       (font
         (size 1.27 1.27))))
-  (property "Footprint" "pulsarfab:USB_A_GCT_USB1046_Edge"
+  (property "Footprint" "pulsarfab:USB_A_SHOUHAN_AF90ZJWG_THT"
     (at 243.84 99.06 0.0)
     (effects
@@
         (size 1.27 1.27))
       (hide yes)))
-  (property "Datasheet" "https://datasheet.lcsc.com/datasheet/pdf/69cc4fb97da31d4274b463dbae6ae45e.pdf?productCode=C6307429"
+  (property "Datasheet" "https://datasheet.lcsc.com/datasheet/pdf/13e3587bf595c7e2c810c5f268cf321c.pdf?productCode=C456019"
     (at 243.84 99.06 0.0)
     (effects
@@
         (size 1.27 1.27))
       (hide yes)))
-  (property "LCSC" "C6307429"
+  (property "LCSC" "C456019"
     (at 243.84 99.06 0.0)
     (effects
@@
         (size 1.27 1.27))
       (hide yes)))
-  (property "MPN" "USB1046-GF-0190-L-B-A"
+  (property "MPN" "AF 90 ZJWG"
     (at 243.84 99.06 0.0)
     (effects
@@
         (size 1.27 1.27))
       (hide yes)))
-  (property "Manufacturer" "Global Connector Technology"
+  (property "Manufacturer" "SHOU HAN"
     (at 243.84 99.06 0.0)
     (effects

Commit message: Reduce PulsarPower power-path cost while retaining current monitoring
Other:
- title: PulsarDew Hub - USB 2.0 downstream port -> PulsarPower - USB 2.0 downstream port
Changed lines of the file:
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@@
 (kicad_sch (version 20260306) (generator "eeschema") (generator_version "10.0") (paper "A4")
-(title_block (title "PulsarDew Hub - USB 2.0 downstream port") (date "2026-10-03") (rev "0.2-draft") (company "PulsarFab"))
+(title_block (title "PulsarPower - USB 2.0 downstream port") (date "2026-10-03") (rev "0.3-draft") (company "PulsarFab"))
 (text "USB DOWNSTREAM | 500 mA service | independent power and overcurrent" (at 20.3200 16.5100 0) (effects (font (size 1.8 1.8)) (justify left top)))
 (hierarchical_label "V5" (shape input) (at 25.4000 35.5600 0) (effects (font (size 1.27 1.27)) (justify left bottom)))
