File: hardware/pulsardewhub/usb_hub.kicad_sch (KiCad schematic)
At the start: 48 parts, among them J40 USB-C upstream, U40 USB2517-JZX, U41 TPS3808G33DBV, U42 USBLC6-2SC6, Y40 24MHz / CL=12pF

Commit message: Reduce PulsarPower power-path cost while retaining current monitoring
Other:
- title: PulsarDew Hub - USB 2.0 hub and upstream interface -> PulsarPower - USB 2.0 hub and upstream interface
Changed lines of the file:
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@@
 (kicad_sch (version 20260306) (generator "eeschema") (generator_version "10.0") (paper "A2")
-(title_block (title "PulsarDew Hub - USB 2.0 hub and upstream interface") (date "2026-10-03") (rev "0.2-draft") (company "PulsarFab"))
+(title_block (title "PulsarPower - USB 2.0 hub and upstream interface") (date "2026-10-03") (rev "0.3-draft") (company "PulsarFab"))
 (text "USB HUB | USB2517 | internal port 1 + external ports 2-5; ports 6/7 disabled" (at 20.3200 16.5100 0) (effects (font (size 2 2)) (justify left top)))
 (symbol

Commit message: Use stocked HRO USB-C sockets on PulsarPower and PulsarDew
Parts:
- J40: footprint Connector_USB:USB_C_Receptacle_GCT_USB4105-xx-A_16P_TopMnt_Horizontal -> pulsarfab:USB_C_HRO_TYPE-C-31-M-12; LCSC C3020560 -> C165948; MPN USB4105-GF-A -> TYPE-C-31-M-12; Manufacturer Global Connector Technology -> Korean Hroparts Elec
Changed lines of the file:
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@@
       (font
         (size 1.27 1.27))))
-  (property "Footprint" "Connector_USB:USB_C_Receptacle_GCT_USB4105-xx-A_16P_TopMnt_Horizontal"
+  (property "Footprint" "pulsarfab:USB_C_HRO_TYPE-C-31-M-12"
     (at 350.52 66.04 0.0)
     (effects
@@
         (size 1.27 1.27))
       (hide yes)))
-  (property "Datasheet" "https://datasheet.lcsc.com/datasheet/pdf/76718c6dacc0a6125953c12b5ebc82df.pdf?productCode=C3020560"
+  (property "Datasheet" "https://datasheet.lcsc.com/datasheet/pdf/9e56b777c022540fcce7c7f67825f55e.pdf?productCode=C165948"
     (at 350.52 66.04 0.0)
     (effects
@@
         (size 1.27 1.27))
       (hide yes)))
-  (property "LCSC" "C3020560"
+  (property "LCSC" "C165948"
     (at 350.52 66.04 0.0)
     (effects
@@
         (size 1.27 1.27))
       (hide yes)))
-  (property "MPN" "USB4105-GF-A"
+  (property "MPN" "TYPE-C-31-M-12"
     (at 350.52 66.04 0.0)
     (effects
@@
         (size 1.27 1.27))
       (hide yes)))
-  (property "Manufacturer" "Global Connector Technology"
+  (property "Manufacturer" "Korean Hroparts Elec"
     (at 350.52 66.04 0.0)
     (effects
